Commit message: CMake dependency 2023

File: ecn_2023/ecn_2023/urdf/world/world.xacro (robot description, xacro)
@@ -1,8 +1,9 @@
 <?xml version="1.0"?>
-<robot name="world" xmlns:xacro="http://www.ros.org/wiki/xacro">
+<robot name="terrain" xmlns:xacro="http://www.ros.org/wiki/xacro">
   <material name="water">
     <color rgba="0.02 0.26 0.46 0.6"/>
   </material>
-  <link name="world">
+  <link name="world"/>
+  <link name="terrain">
     <visual>
     <geometry>
@@ -20,7 +21,11 @@
     </visual>
   </link>
-  <joint name="surface" type="fixed">
+  <joint name="surface_jnt" type="fixed">
     <parent link="world"/>
     <child link="surface"/>
   </joint>
+  <joint name="terrain_jnt" type="fixed">
+    <parent link="world"/>
+    <child link="terrain"/>
+  </joint>
 </robot>
